File: usb.sch (KiCad schematic (older format))
At the start: 25 parts, among them J4 CONN_02X03, U1 LFE5U-85F-6BG381C, U6 FT231XS, Y1 FNETHE025

Commit message: schematics: connect 25MHz oscillator CLK_OE with FPGA
Connections:
- net labels added: CLK_OE
- wire segments 74 -> 71
Changed lines of the file:
@@
 $EndComp
-Wire Wire Line
-	5450 1150 5450 1200
 Wire Wire Line
 	5300 1450 5200 1450
-Wire Wire Line
-	5200 1450 5200 1200
-Wire Wire Line
-	5200 1200 5450 1200
-Connection ~ 5450 1200
 $Comp
 L power:GND #PWR0110
@@
 	6450 3700 6550 3700
 Wire Wire Line
-	5450 1200 5450 1250
-Wire Wire Line
 	2550 4850 2750 4850
 Wire Wire Line
@@
 Text Notes 7550 2600 0    60   ~ 0
 WIFI_RXD2
+Wire Wire Line
+	5450 1150 5450 1250
+Text GLabel 5200 1450 0    60   Input ~ 0
+CLK_OE
+Text GLabel 10150 2050 2    60   Input ~ 0
+CLK_OE
 $EndSCHEMATC
