File: ulx3s.kicad_pcb (KiCad board)
At the start: 4 copper layers, 172 parts, among them Q2 2N7002, SW1 SW_DIP_x04, U1 LFE5U-85F-6BG381C, U2 MT48LC16M16A2TG, U5 TLV62569DBV, U6 FT231XS, U8 MAX11125, U9 ESP32-WROOM, Y1 FNETHE025, Y2 32768Hz

Commit message: PCB v3.0.9: connect CLK_OE to FPGA
Connections:
- AUDIO1 pad 5: Net-(AUDIO1-Pad5) -> (no net)
- AUDIO1 pad 6: Net-(AUDIO1-Pad6) -> (no net)
- U1 pad A15: Net-(U1-PadA15) -> (no net)
- U1 pad C9: Net-(U1-PadC9) -> (no net)
- U1 pad D10: Net-(U1-PadD10) -> (no net)
- U1 pad D11: Net-(U1-PadD11) -> (no net)
- U1 pad D12: Net-(U1-PadD12) -> (no net)
- U1 pad D9: Net-(U1-PadD9) -> (no net)
- U1 pad E10: Net-(U1-PadE10) -> (no net)
- U1 pad E11: Net-(U1-PadE11) -> (no net)
- U1 pad E6: Net-(U1-PadE6) -> (no net)
- U1 pad E9: Net-(U1-PadE9) -> (no net)
- U1 pad J4: Net-(U1-PadJ4) -> (no net)
- U1 pad J5: Net-(U1-PadJ5) -> (no net)
- U1 pad K16: Net-(U1-PadK16) -> (no net)
- U1 pad K17: Net-(U1-PadK17) -> (no net)
- U1 pad K5: Net-(U1-PadK5) -> CLK_OE
- U1 pad M5: Net-(U1-PadM5) -> (no net)
- U1 pad N5: SD_CD -> (no net)
- U1 pad P5: SD_WP -> (no net)
- U1 pad R3: Net-(U1-PadR3) -> (no net)
- U1 pad T16: Net-(U1-PadT16) -> (no net)
- U1 pad W13: Net-(U1-PadW13) -> (no net)
- U1 pad W14: Net-(U1-PadW14) -> (no net)
- U1 pad W17: Net-(U1-PadW17) -> (no net)
- U1 pad W18: Net-(U1-PadW18) -> (no net)
- U1 pad W4: Net-(U1-PadW4) -> (no net)
- U1 pad W5: Net-(U1-PadW5) -> (no net)
- U1 pad W8: Net-(U1-PadW8) -> (no net)
- U1 pad W9: Net-(U1-PadW9) -> (no net)
- U8 pad 12: Net-(U8-Pad12) -> (no net)
- U8 pad 25: Net-(U8-Pad25) -> (no net)
- U9 pad 12: Net-(U9-Pad12) -> (no net)
- U9 pad 17: Net-(U9-Pad17) -> (no net)
- U9 pad 18: Net-(U9-Pad18) -> (no net)
- U9 pad 19: Net-(U9-Pad19) -> (no net)
- U9 pad 20: Net-(U9-Pad20) -> (no net)
- U9 pad 21: Net-(U9-Pad21) -> (no net)
- U9 pad 22: Net-(U9-Pad22) -> (no net)
- U9 pad 32: Net-(U9-Pad32) -> (no net)
- U9 pad 4: Net-(U9-Pad4) -> (no net)
- U9 pad 5: Net-(U9-Pad5) -> (no net)
- US1 pad 4: Net-(US1-Pad4) -> (no net)
- Y1 pad 1: +3V3 -> CLK_OE
- Y2 pad 2: Net-(Y2-Pad2) -> (no net)
- Y2 pad 3: Net-(Y2-Pad3) -> (no net)
